File: Kicad/RTO_cart.kicad_sch (KiCad schematic)
At the start: 17 parts, among them J1 2x22 card edge connector, J2 Oled 0.91" female, SW1 SW_Push, SW2 SW_Push, U1 74LVC245, U2 74LVC245, U3 74LVC245, U4 Teensy4.1

Commit message: Add files via upload
Parts:
- added C4: 100nF, Capacitor_THT:C_Disc_D3.8mm_W2.6mm_P2.50mm, symbol Device:C
- added R5: 1K, Resistor_THT:R_Axial_DIN0204_L3.6mm_D1.6mm_P7.62mm_Horizontal, symbol Device:R
- added R6: 4K7, Resistor_THT:R_Axial_DIN0204_L3.6mm_D1.6mm_P7.62mm_Horizontal, symbol Device:R
- added SW3: SW_Push, Button_Switch_THT:SW_PUSH_6mm, symbol Switch:SW_Push
- added U5: 74LVC245, Package_DIP:DIP-20_W7.62mm_Socket, symbol 74xx:74LS245
Connections:
- net +3.3V: now also C1.1, C2.1, C3.1, C4.1, R5.2, U5.20 (VCC)
- net +5V: no longer C1.1, C2.1, C3.1
- net GND: now also J1.10 (Pin_10), J1.8 (Pin_8), C4.2, R6.2, U5.10 (GND), U5.19 (CE); no longer J1.12 (Pin_12)
- net ~{msync'}: now reaches J1.3 (Pin_3)
- net ~{msync'}: now also U3.15 (B3)
- net ~{MSYNC}: now reaches U3.5 (A3)
- net ~{MSYNC}: now also U4.10 (8_TX2_IN1)
- net BT3: now reaches U4.26 (34_RX8)
- net BT3: now also SW3.1
- net DIR2: now reaches U4.8 (6_OUT1D)
- net DIR2: now also U5.1 (A->B)
- net RST: now reaches U4.9 (7_RX2_OUT1A)
- net RST: now also U5.2 (A0)
- new net: R5.1, SW3.2
- new net rst': J1.12 (Pin_12), R6.1, U5.18 (B0)
- no-connect marks 56 -> 61
Other:
- company: (none) -> Andrea Ottaviani
- title: (none) -> RTO-Multicart
- moved on the sheet: J2

Commit message: Add files via upload
Parts:
- removed C4: 100nF, Capacitor_THT:C_Disc_D3.8mm_W2.6mm_P2.50mm, symbol Device:C
- removed R5: 1K, Resistor_THT:R_Axial_DIN0204_L3.6mm_D1.6mm_P7.62mm_Horizontal, symbol Device:R
- removed R6: 4K7, Resistor_THT:R_Axial_DIN0204_L3.6mm_D1.6mm_P7.62mm_Horizontal, symbol Device:R
- removed SW3: SW_Push, Button_Switch_THT:SW_PUSH_6mm, symbol Switch:SW_Push
- removed U5: 74LVC245, Package_DIP:DIP-20_W7.62mm_Socket, symbol 74xx:74LS245
- U1, U2, U3: value 74LVC245 -> 74LS245
Connections:
- net rst' is gone; now on net GND: J1.12 (Pin_12)
- net +3.3V: no longer C1.1, C2.1, C3.1
- net +5V: now also C1.1, C2.1, C3.1
- net GND: no longer J1.10 (Pin_10), J1.8 (Pin_8)
- net BT3: no longer names the net of U4.26 (34_RX8)
- net DIR2: no longer names the net of U4.8 (6_OUT1D)
- net RST: no longer names the net of U4.9 (7_RX2_OUT1A)
- net ~{MSYNC}: no longer names the net of U3.5 (A3)
- net ~{MSYNC}: no longer U4.10 (8_TX2_IN1)
- net ~{msync'}: no longer names the net of J1.3 (Pin_3)
- net ~{msync'}: no longer U3.15 (B3)
- no-connect marks 61 -> 56
Other:
- company: Andrea Ottaviani -> (none)
- title: RTO-Multicart -> (none)
- moved on the sheet: J2

Commit message: Add files via upload
corrected the level shifter ICs to 74LVC245 instead of wrong typed 74LS245: WARNING! use only 74LVC245 chips, the other types could damage your Teensy becouse they output 5V instead of 3V3!
Parts:
- U1, U2, U3: value 74LS245 -> 74LVC245
Changed lines of the file:
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@@
       (effects (font (size 1.27 1.27)) (justify left))
     )
-    (property "Value" "74LS245" (id 1) (at 187.4394 31.8571 0)
+    (property "Value" "74LVC245" (id 1) (at 187.4394 31.8571 0)
       (effects (font (size 1.27 1.27)) (justify left))
     )
@@
       (effects (font (size 1.27 1.27)) hide)
     )
-    (property "Datasheet" "http://www.ti.com/lit/gpn/sn74LS245" (id 3) (at 185.42 48.26 0)
+    (property "Datasheet" "" (id 3) (at 185.42 48.26 0)
       (effects (font (size 1.27 1.27)) hide)
     )
@@
       (effects (font (size 1.27 1.27)) (justify left))
     )
-    (property "Value" "74LS245" (id 1) (at 97.2694 31.8571 0)
+    (property "Value" "74LVC245" (id 1) (at 97.2694 31.8571 0)
       (effects (font (size 1.27 1.27)) (justify left))
     )
@@
       (effects (font (size 1.27 1.27)) hide)
     )
-    (property "Datasheet" "http://www.ti.com/lit/gpn/sn74LS245" (id 3) (at 95.25 48.26 0)
+    (property "Datasheet" "" (id 3) (at 95.25 48.26 0)
       (effects (font (size 1.27 1.27)) hide)
     )
@@
       (effects (font (size 1.27 1.27)) (justify left))
     )
-    (property "Value" "74LS245" (id 1) (at 141.7194 31.8571 0)
+    (property "Value" "74LVC245" (id 1) (at 141.7194 31.8571 0)
       (effects (font (size 1.27 1.27)) (justify left))
     )
@@
       (effects (font (size 1.27 1.27)) hide)
     )
-    (property "Datasheet" "http://www.ti.com/lit/gpn/sn74LS245" (id 3) (at 139.7 48.26 0)
+    (property "Datasheet" "" (id 3) (at 139.7 48.26 0)
       (effects (font (size 1.27 1.27)) hide)
     )
@@
     )
     (path "/697b2099-5d1e-421b-86fb-66456fe646ee"
-      (reference "U1") (unit 1) (value "74LS245") (footprint "Package_DIP:DIP-20_W7.62mm_Socket")
+      (reference "U1") (unit 1) (value "74LVC245") (footprint "Package_DIP:DIP-20_W7.62mm_Socket")
     )
     (path "/6be8ebdc-952c-4ab9-8e80-82974edcb5f0"
-      (reference "U2") (unit 1) (value "74LS245") (footprint "Package_DIP:DIP-20_W7.62mm_Socket")
+      (reference "U2") (unit 1) (value "74LVC245") (footprint "Package_DIP:DIP-20_W7.62mm_Socket")
     )
     (path "/678e113b-998d-4fc9-b7c0-b0cd26248191"
-      (reference "U3") (unit 1) (value "74LS245") (footprint "Package_DIP:DIP-20_W7.62mm_Socket")
+      (reference "U3") (unit 1) (value "74LVC245") (footprint "Package_DIP:DIP-20_W7.62mm_Socket")
     )
     (path "/b76b3bdd-28ec-4a43-a3e2-5a3321ec7e57"
