File: ver1.1a-beta/kicad/RTO_cart.kicad_pcb (KiCad board)
At the start: 2 copper layers, 68.1 x 90.1 mm, 22 parts, among them J1 2x22 card edge connector, J2 Oled 0.91" female, SW1 SW_Push, SW2 SW_Push, SW3 SW_Push, U1 74LVC245, U2 74LVC245, U3 74LVC245, U4 Teensy4.1, U5 74LVC245

Commit message: Add files via upload
Connections:
- J1 pad 3: unconnected-(J1-Pad3) -> ~{msync'}
- U3 pad 15: unconnected-(U3-Pad15) -> ~{msync'}
- U3 pad 5: unconnected-(U3-Pad5) -> ~{MSYNC}
- U4 pad 10: unconnected-(U4-Pad10) -> ~{MSYNC}
Routing:
- net ~{MSYNC}: track 0.00 -> 49.8 mm
- net bdir': track 53.7 -> 102.5 mm
- net ~{msync'}: track 0.00 -> 46.5 mm
- net d0': track 71.3 -> 40.9 mm, vias 0 -> 1
- net +5V: track 96.3 -> 116.2 mm, vias 2 -> 0
- net D15: track 61.6 -> 78.3 mm
- net d8': track 65.3 -> 81.9 mm, vias 0 -> 2
- net D14: track 73.6 -> 61.1 mm, vias 1 -> 0
- net d15': track 37.3 -> 25.9 mm
- net D10: track 59.1 -> 48.4 mm
- net D0: track 33.7 -> 43.7 mm
- net DIR: track 72.3 -> 63.3 mm
- net GND: track 360.3 -> 368.8 mm
- net BC2: track 57.6 -> 49.3 mm, vias 0 -> 1
- net BC1: track 54.6 -> 47.7 mm, vias 0 -> 1
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Other:
- board text added: "RTO Cart by A.Ottaviani v.1.1a (28/1/2023)"
- board text removed: "RTO Cart by A.Ottaviani v.1.1a (25/1/2023)"
