File: ver1.1a-beta/kicad/RTO_cart.kicad_sch (KiCad schematic)
At the start: 22 parts, among them J1 2x22 card edge connector, J2 Oled 0.91" female, SW1 SW_Push, SW2 SW_Push, SW3 SW_Push, U1 74LVC245, U2 74LVC245, U3 74LVC245, U4 Teensy4.1, U5 74LVC245

Commit message: Add files via upload
Connections:
- net ~{msync'}: now reaches J1.3 (Pin_3)
- net ~{msync'}: now also U3.15 (B3)
- net ~{MSYNC}: now reaches U3.5 (A3)
- net ~{MSYNC}: now also U4.10 (8_TX2_IN1)
- no-connect marks 65 -> 61
Changed lines of the file:
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@@
   (no_connect (at 125.73 129.54))
   (no_connect (at 125.73 154.94))
-  (no_connect (at 69.85 119.38))
   (no_connect (at 69.85 121.92))
   (no_connect (at 69.85 124.46))
@@
   (no_connect (at 69.85 147.32))
   (no_connect (at 69.85 149.86))
-  (no_connect (at 198.12 43.18))
-  (no_connect (at 172.72 43.18))
   (no_connect (at 49.53 64.77))
   (no_connect (at 247.65 53.34))
@@
   (no_connect (at 198.12 50.8))
   (no_connect (at 198.12 53.34))
-  (no_connect (at 36.83 31.75))
   (no_connect (at 222.25 53.34))
   (no_connect (at 125.73 92.71))
@@
     )
   )
+  (global_label "~{MSYNC}" (shape input) (at 69.85 119.38 180) (fields_autoplaced)
+    (effects (font (size 1.27 1.27)) (justify right))
+    (property "Intersheet References" "${INTERSHEET_REFS}" (id 0) (at 61.0869 119.3006 0)
+      (effects (font (size 1.27 1.27)) (justify right) hide)
+    )
+  )
   (global_label "BT2" (shape input) (at 153.67 104.14 180) (fields_autoplaced)
     (effects (font (size 1.27 1.27)) (justify right))
@@
     )
   )
+  (global_label "~{MSYNC}" (shape input) (at 172.72 43.18 180) (fields_autoplaced)
+    (effects (font (size 1.27 1.27)) (justify right))
+    (property "Intersheet References" "${INTERSHEET_REFS}" (id 0) (at 163.9569 43.1006 0)
+      (effects (font (size 1.27 1.27)) (justify right) hide)
+    )
+  )
   (global_label "d5'" (shape input) (at 36.83 44.45 180) (fields_autoplaced)
     (effects (font (size 1.27 1.27)) (justify right))
@@
     )
   )
+  (global_label "~{msync'}" (shape input) (at 36.83 31.75 180) (fields_autoplaced)
+    (effects (font (size 1.27 1.27)) (justify right))
+    (property "Intersheet References" "${INTERSHEET_REFS}" (id 0) (at 27.8855 31.8294 0)
+      (effects (font (size 1.27 1.27)) (justify right) hide)
+    )
+  )
   (global_label "D3" (shape input) (at 107.95 43.18 0) (fields_autoplaced)
     (effects (font (size 1.27 1.27)) (justify left))
@@
     )
   )
+  (global_label "~{msync'}" (shape input) (at 198.12 43.18 0) (fields_autoplaced)
+    (effects (font (size 1.27 1.27)) (justify left))
+    (property "Intersheet References" "${INTERSHEET_REFS}" (id 0) (at 207.0645 43.1006 0)
+      (effects (font (size 1.27 1.27)) (justify left) hide)
+    )
+  )
